Commit message: Add gladlaks visuals

File: gladlaks_description/urdf/base.xacro (robot description, xacro)
@@ -23,5 +23,5 @@
     Open the meshes for the RexROV vehicle in Blender to see an example on the mesh placement.
   -->
-  <xacro:property name="visual_mesh_file" value="file://$(find gladlaks_description)/meshes/manta_shell.dae"/>
+  <xacro:property name="visual_mesh_file" value="file://$(find gladlaks_description)/meshes/Gladlaks_centered_body.dae"/>
   <!-- Collision geometry mesh, usually in STL format (it is recommended to keep
   this geometry as simple as possible to improve the performance the physics engine
@@ -46,5 +46,5 @@
           <origin xyz="0 0 0" rpy="0 0 0"/>
           <geometry>
-            <mesh filename="${visual_mesh_file}" scale="1 1 1" />
+            <mesh filename="${visual_mesh_file}" scale="0.01 0.01 0.01" />
           </geometry>
         </visual>
