Commit message: Further development

File: gladlaks_description/robots/default.xacro (robot description, xacro)
@@ -3,5 +3,5 @@
   <xacro:arg name="debug" default="0"/>
   <xacro:arg name="namespace" default="gladlaks"/>
-  <xacro:arg name="inertial_reference_frame" default="world_ned"/>
+  <xacro:arg name="inertial_reference_frame" default="world"/>
   <!-- Download gladlaks parameters -->
   <xacro:property name="gladlaks_yaml_file" value="$(find gladlaks_description)/config/gladlaks.yaml" />

File: gladlaks_description/urdf/base.xacro (robot description, xacro)
@@ -23,5 +23,5 @@
     Open the meshes for the RexROV vehicle in Blender to see an example on the mesh placement.
   -->
-  <xacro:property name="visual_mesh_file" value="file://$(find gladlaks_description)/meshes/Gladlaks_centered_body.dae"/>
+  <xacro:property name="visual_mesh_file" value="file://$(find gladlaks_description)/meshes/manta_shell.dae"/>
   <!-- Collision geometry mesh, usually in STL format (it is recommended to keep
   this geometry as simple as possible to improve the performance the physics engine

Commit message: Fix visual and add parameters

File: gladlaks_description/robots/default.xacro (robot description, xacro)
@@ -4,7 +4,7 @@
   <xacro:arg name="namespace" default="gladlaks"/>
   <xacro:arg name="inertial_reference_frame" default="world"/>
-  <!-- Download gladlaks parameters -->
-  <xacro:property name="gladlaks_yaml_file" value="$(find gladlaks_description)/config/gladlaks.yaml" />
-  <xacro:property name="props" value="${load_yaml(gladlaks_yaml_file)}"/>
+  <xacro:arg name="param_file" default="$(find gladlaks_description)/config/gladlaks.yaml"/>
+  <xacro:property name="param_file" value="$(arg param_file)" />
+  <xacro:property name="props" value="${load_yaml(param_file)}"/>
   <!-- Include the ROV macro file -->
   <xacro:include filename="$(find gladlaks_description)/urdf/base.xacro"/>

File: gladlaks_description/urdf/base.xacro (robot description, xacro)
@@ -46,5 +46,5 @@
           <origin xyz="0 0 0" rpy="0 0 0"/>
           <geometry>
-            <mesh filename="${visual_mesh_file}" scale="0.01 0.01 0.01" />
+            <mesh filename="${visual_mesh_file}" scale="0.011 0.011 0.011" />
           </geometry>
         </visual>
